Commit message: kitchen mesh path

File: notebooks/dlr_kitchen.urdf (robot description, URDF)
Before this commit: robot dlr_kitchen, 21 links, 20 joints
Links:
- link drawer_01: geometry collision mesh filename=~/workspace/ros/src/dlr_kitchen/dlr_kitchen/dlr_kitchen/mes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 scale=1.0 1.0 1.0; collision mesh filename=~/workspace/ros/src/dlr_kitchen/dlr_kitchen/dlr_kitchen/mes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 scale=1.0 1.0 1.0
- link drawer_01_handle: geometry collision mesh filename=~/workspace/ros/src/dlr_kitchen/dlr_kitchen/dlr_kitchen/mes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 scale=1.0 1.0 1.0; collision mesh filename=~/workspace/ros/src/dlr_kitchen/dlr_kitchen/dlr_kitchen/mes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 scale=1.0 1.0 1.0
- link drawer_02: geometry collision mesh filename=~/workspace/ros/src/dlr_kitchen/dlr_kitchen/dlr_kitchen/mes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 scale=1.0 1.0 1.0; collision mesh filename=~/workspace/ros/src/dlr_kitchen/dlr_kitchen/dlr_kitchen/mes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 scale=1.0 1.0 1.0
- link drawer_02_handle: geometry collision mesh filename=~/workspace/ros/src/dlr_kitchen/dlr_kitchen/dlr_kitchen/mes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 scale=1.0 1.0 1.0; collision mesh filename=~/workspace/ros/src/dlr_kitchen/dlr_kitchen/dlr_kitchen/mes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 scale=1.0 1.0 1.0
- link drawer_03: geometry collision mesh filename=~/workspace/ros/src/dlr_kitchen/dlr_kitchen/dlr_kitchen/mes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 scale=1.0 1.0 1.0; collision mesh filename=~/workspace/ros/src/dlr_kitchen/dlr_kitchen/dlr_kitchen/mes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 scale=1.0 1.0 1.0
- link drawer_03_handle: geometry collision mesh filename=~/workspace/ros/src/dlr_kitchen/dlr_kitchen/dlr_kitchen/mes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 scale=1.0 1.0 1.0; collision mesh filename=~/workspace/ros/src/dlr_kitchen/dlr_kitchen/dlr_kitchen/mes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 scale=1.0 1.0 1.0
- link drawer_04: geometry collision mesh filename=~/workspace/ros/src/dlr_kitchen/dlr_kitchen/dlr_kitchen/mes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 scale=1.0 1.0 1.0; collision mesh filename=~/workspace/ros/src/dlr_kitchen/dlr_kitchen/dlr_kitchen/mes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 scale=1.0 1.0 1.0
- link drawer_04_handle: geometry collision mesh filename=~/workspace/ros/src/dlr_kitchen/dlr_kitchen/dlr_kitchen/mes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 scale=1.0 1.0 1.0; collision mesh filename=~/workspace/ros/src/dlr_kitchen/dlr_kitchen/dlr_kitchen/mes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 scale=1.0 1.0 1.0
- link drawer_05: geometry collision mesh filename=~/workspace/ros/src/dlr_kitchen/dlr_kitchen/dlr_kitchen/mes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 scale=1.0 1.0 1.0; collision mesh filename=~/workspace/ros/src/dlr_kitchen/dlr_kitchen/dlr_kitchen/mes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 scale=1.0 1.0 1.0
- link drawer_05_handle: geometry collision mesh filename=~/workspace/ros/src/dlr_kitchen/dlr_kitchen/dlr_kitchen/mes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 scale=1.0 1.0 1.0; collision mesh filename=~/workspace/ros/src/dlr_kitchen/dlr_kitchen/dlr_kitchen/mes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 scale=1.0 1.0 1.0
- link drawer_06: geometry collision mesh filename=~/workspace/ros/src/dlr_kitchen/dlr_kitchen/dlr_kitchen/mes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 scale=1.0 1.0 1.0; collision mesh filename=~/workspace/ros/src/dlr_kitchen/dlr_kitchen/dlr_kitchen/mes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 scale=1.0 1.0 1.0
- link drawer_06_handle: geometry collision mesh filename=~/workspace/ros/src/dlr_kitchen/dlr_kitchen/dlr_kitchen/mes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 scale=1.0 1.0 1.0; collision mesh filename=~/workspace/ros/src/dlr_kitchen/dlr_kitchen/dlr_kitchen/mes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 scale=1.0 1.0 1.0
- link fridge: geometry collision mesh filename=~/workspace/ros/src/dlr_kitchen/dlr_kitchen/dlr_kitchen/mes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 scale=1.0 1.0 1.0; collision mesh filename=~/workspace/ros/src/dlr_kitchen/dlr_kitchen/dlr_kitchen/mes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 scale=1.0 1.0 1.0
- link fridge_door: geometry collision mesh filename=~/workspace/ros/src/dlr_kitchen/dlr_kitchen/dlr_kitchen/mes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 scale=1.0 1.0 1.0; visual mesh filename=~/workspace/ros/src/dlr_kitchen/dlr_kitchen/dlr_kitchen/mes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 scale=1.0 1.0 1.0
- link fridge_door_handle: geometry collision mesh filename=~/workspace/ros/src/dlr_kitchen/dlr_kitchen/dlr_kitchen/mes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 scale=1.0 1.0 1.0; collision mesh filename=~/workspace/ros/src/dlr_kitchen/dlr_kitchen/dlr_kitchen/mes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 scale=1.0 1.0 1.0
- link kitchenette: geometry collision mesh filename=~/workspace/ros/src/dlr_kitchen/dlr_kitchen/dlr_kitchen/mes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 scale=1.0 1.0 1.0; collision mesh filename=~/workspace/ros/src/dlr_kitchen/dlr_kitchen/dlr_kitchen/mes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 scale=1.0 1.0 1.0
- link oven_door: geometry collision mesh filename=~/workspace/ros/src/dlr_kitchen/dlr_kitchen/dlr_kitchen/mes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 scale=1.0 1.0 1.0; visual mesh filename=~/workspace/ros/src/dlr_kitchen/dlr_kitchen/dlr_kitchen/mes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 scale=1.0 1.0 1.0
- link oven_door_handle: geometry collision mesh filename=~/workspace/ros/src/dlr_kitchen/dlr_kitchen/dlr_kitchen/mes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 scale=1.0 1.0 1.0; collision mesh filename=~/workspace/ros/src/dlr_kitchen/dlr_kitchen/dlr_kitchen/mes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 scale=1.0 1.0 1.0
- link oven_drawer: geometry collision mesh filename=~/workspace/ros/src/dlr_kitchen/dlr_kitchen/dlr_kitchen/mes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 scale=1.0 1.0 1.0; collision mesh filename=~/workspace/ros/src/dlr_kitchen/dlr_kitchen/dlr_kitchen/mes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 scale=1.0 1.0 1.0
- link oven_drawer_handle: geometry collision mesh filename=~/workspace/ros/src/dlr_kitchen/dlr_kitchen/dlr_kitchen/mes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 scale=1.0 1.0 1.0; collision mesh filename=~/workspace/ros/src/dlr_kitchen/dlr_kitchen/dlr_kitchen/mes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 scale=1.0 1.0 1.0

Commit message: kitchen mesh path

File: notebooks/dlr_kitchen.urdf (robot description, URDF)
Before this commit: robot dlr_kitchen, 21 links, 20 joints
Links:
- link drawer_01: geometry collision mesh filename=/home/jovyan/workspace/ros/src/dlr_kitchen/dlr_kitchen/dlr_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 scale=1.0 1.0 1.0; collision mesh filename=/home/jovyan/workspace/ros/src/dlr_kitchen/dlr_kitchen/dlr_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 scale=1.0 1.0 1.0
- link drawer_01_handle: geometry collision mesh filename=/home/jovyan/workspace/ros/src/dlr_kitchen/dlr_kitchen/dlr_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 scale=1.0 1.0 1.0; collision mesh filename=/home/jovyan/workspace/ros/src/dlr_kitchen/dlr_kitchen/dlr_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 scale=1.0 1.0 1.0
- link drawer_02: geometry collision mesh filename=/home/jovyan/workspace/ros/src/dlr_kitchen/dlr_kitchen/dlr_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 scale=1.0 1.0 1.0; collision mesh filename=/home/jovyan/workspace/ros/src/dlr_kitchen/dlr_kitchen/dlr_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 scale=1.0 1.0 1.0
- link drawer_02_handle: geometry collision mesh filename=/home/jovyan/workspace/ros/src/dlr_kitchen/dlr_kitchen/dlr_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 scale=1.0 1.0 1.0; collision mesh filename=/home/jovyan/workspace/ros/src/dlr_kitchen/dlr_kitchen/dlr_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 scale=1.0 1.0 1.0
- link drawer_03: geometry collision mesh filename=/home/jovyan/workspace/ros/src/dlr_kitchen/dlr_kitchen/dlr_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 scale=1.0 1.0 1.0; collision mesh filename=/home/jovyan/workspace/ros/src/dlr_kitchen/dlr_kitchen/dlr_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 scale=1.0 1.0 1.0
- link drawer_03_handle: geometry collision mesh filename=/home/jovyan/workspace/ros/src/dlr_kitchen/dlr_kitchen/dlr_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 scale=1.0 1.0 1.0; collision mesh filename=/home/jovyan/workspace/ros/src/dlr_kitchen/dlr_kitchen/dlr_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 scale=1.0 1.0 1.0
- link drawer_04: geometry collision mesh filename=/home/jovyan/workspace/ros/src/dlr_kitchen/dlr_kitchen/dlr_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 scale=1.0 1.0 1.0; collision mesh filename=/home/jovyan/workspace/ros/src/dlr_kitchen/dlr_kitchen/dlr_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 scale=1.0 1.0 1.0
- link drawer_04_handle: geometry collision mesh filename=/home/jovyan/workspace/ros/src/dlr_kitchen/dlr_kitchen/dlr_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 scale=1.0 1.0 1.0; collision mesh filename=/home/jovyan/workspace/ros/src/dlr_kitchen/dlr_kitchen/dlr_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 scale=1.0 1.0 1.0
- link drawer_05: geometry collision mesh filename=/home/jovyan/workspace/ros/src/dlr_kitchen/dlr_kitchen/dlr_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 scale=1.0 1.0 1.0; collision mesh filename=/home/jovyan/workspace/ros/src/dlr_kitchen/dlr_kitchen/dlr_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 scale=1.0 1.0 1.0
- link drawer_05_handle: geometry collision mesh filename=/home/jovyan/workspace/ros/src/dlr_kitchen/dlr_kitchen/dlr_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 scale=1.0 1.0 1.0; collision mesh filename=/home/jovyan/workspace/ros/src/dlr_kitchen/dlr_kitchen/dlr_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 scale=1.0 1.0 1.0
- link drawer_06: geometry collision mesh filename=/home/jovyan/workspace/ros/src/dlr_kitchen/dlr_kitchen/dlr_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 scale=1.0 1.0 1.0; collision mesh filename=/home/jovyan/workspace/ros/src/dlr_kitchen/dlr_kitchen/dlr_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 scale=1.0 1.0 1.0
- link drawer_06_handle: geometry collision mesh filename=/home/jovyan/workspace/ros/src/dlr_kitchen/dlr_kitchen/dlr_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 scale=1.0 1.0 1.0; collision mesh filename=/home/jovyan/workspace/ros/src/dlr_kitchen/dlr_kitchen/dlr_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 scale=1.0 1.0 1.0
- link fridge: geometry collision mesh filename=/home/jovyan/workspace/ros/src/dlr_kitchen/dlr_kitchen/dlr_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 scale=1.0 1.0 1.0; collision mesh filename=/home/jovyan/workspace/ros/src/dlr_kitchen/dlr_kitchen/dlr_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 scale=1.0 1.0 1.0
- link fridge_door: geometry collision mesh filename=/home/jovyan/workspace/ros/src/dlr_kitchen/dlr_kitchen/dlr_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 scale=1.0 1.0 1.0; visual mesh filename=/home/jovyan/workspace/ros/src/dlr_kitchen/dlr_kitchen/dlr_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 scale=1.0 1.0 1.0
- link fridge_door_handle: geometry collision mesh filename=/home/jovyan/workspace/ros/src/dlr_kitchen/dlr_kitchen/dlr_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 scale=1.0 1.0 1.0; collision mesh filename=/home/jovyan/workspace/ros/src/dlr_kitchen/dlr_kitchen/dlr_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 scale=1.0 1.0 1.0
- link kitchenette: geometry collision mesh filename=/home/jovyan/workspace/ros/src/dlr_kitchen/dlr_kitchen/dlr_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 scale=1.0 1.0 1.0; collision mesh filename=/home/jovyan/workspace/ros/src/dlr_kitchen/dlr_kitchen/dlr_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 scale=1.0 1.0 1.0
- link oven_door: geometry collision mesh filename=/home/jovyan/workspace/ros/src/dlr_kitchen/dlr_kitchen/dlr_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 scale=1.0 1.0 1.0; visual mesh filename=/home/jovyan/workspace/ros/src/dlr_kitchen/dlr_kitchen/dlr_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 scale=1.0 1.0 1.0
- link oven_door_handle: geometry collision mesh filename=/home/jovyan/workspace/ros/src/dlr_kitchen/dlr_kitchen/dlr_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 scale=1.0 1.0 1.0; collision mesh filename=/home/jovyan/workspace/ros/src/dlr_kitchen/dlr_kitchen/dlr_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 scale=1.0 1.0 1.0
- link oven_drawer: geometry collision mesh filename=/home/jovyan/workspace/ros/src/dlr_kitchen/dlr_kitchen/dlr_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 scale=1.0 1.0 1.0; collision mesh filename=/home/jovyan/workspace/ros/src/dlr_kitchen/dlr_kitchen/dlr_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 scale=1.0 1.0 1.0
- link oven_drawer_handle: geometry collision mesh filename=/home/jovyan/workspace/ros/src/dlr_kitchen/dlr_kitchen/dlr_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 scale=1.0 1.0 1.0; collision mesh filename=/home/jovyan/workspace/ros/src/dlr_kitchen/dlr_kitchen/dlr_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 scale=1.0 1.0 1.0
